File: schematic-design/MIDI and Voltage reg.kicad_sch (KiCad schematic)
At the start: 16 parts, among them J1 POWER Barrel Jack, J2 DIN-5_180degree, J3 DIN-5_180degree, U1 6N138 Optocoupler, U2 LM2574Y-5 Buck converter, U3 74LS04

Commit message: Update schematic
Parts:
- added C1, C2: 22pF, symbol Device:C
- added J4: Conn_01x03_Pin, symbol Connector:Conn_01x03_Pin
- added U1: ATmega328P-P, Package_DIP:DIP-28_W7.62mm, symbol MCU_Microchip_ATmega:ATmega328P-P
- added Y1: Crystal, symbol Device:Crystal
Connections:
- net +12V: now also J4.1 (Pin_1)
- net +5V: now also U1.20 (AVCC), U1.7 (VCC); no longer J2.4, R2.2
- net GND: now also J1.MP (MountPin), C1.1, C2.2, J4.3 (Pin_3), U1.22 (GND), U1.8 (GND)
- net UART renamed MIDI IN
- net MIDI IN: now also U1.14 (PB0)
- new net: J2.4, R2.2
- new net: C1.2, U1.9 (XTAL1/PB6), Y1.1
- new net: C2.1, U1.10 (XTAL2/PB7), Y1.2
- new net LED DATA: J4.2 (Pin_2), U1.15 (PB1)
- no-connect marks 0 -> 25
Other:
- note added: "Crytal Oscillator"
- note added: "LED Connector"
- note added: "MIDI Input"
- note added: "MIDI THRU"
- note added: "Microcontroller"
- note added: "Power regulator"
- title: (none) -> MIDI Visualiser
- moved on the sheet: J3, R1, R5, U3A, U3B
