File: pcb-design/Practical Electronics WS2023/Practical Electronics WS2023.kicad_pcb (KiCad board)
At the start: 2 copper layers, 69 parts, among them IC1 SN74HCT04DR, J1 PWR Jack, J2 MIDI Input, J3 MIDI Thru out, J4 Conn_01x03, J5 ISP, J6 Switch connector, J7 Switch connector, J8 Switch connector, U1 6N138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

Commit message: PCB WIP
Parts:
- IC1: value SN74HCT04DR -> NOT GATES N74HCT04DR
- J4: value Conn_01x03 -> LED Connector Conn_01x03
- U1: value 6N138 -> 6N138 Optocoupler
- U2: value ADP2303ARDZ-5.0 -> Convertor ADP2303ARDZ-5.0
- moved D9 111.1 mm to (211.7, 25.3), turned to 90 degrees
- moved C19 101.1 mm to (205.6, 26.4), turned to 90 degrees
- moved J3 99.9 mm to (110.7, 46.0), turned to 180 degrees
- moved D5 90.1 mm to (180.8, 109.2), turned to 90 degrees
- moved C18 88.0 mm to (174.8, 110.5), turned to 90 degrees
- moved J5 87.8 mm to (116.3, 76.7), turned to -90 degrees
- moved D7 84.9 mm to (165.6, 109.8), turned to 90 degrees
- moved C11 82.8 mm to (159.3, 106.0), turned to 90 degrees
- moved C3 81.3 mm to (105.1, 69.4)
- moved C7 81.3 mm to (120.7, 57.2)
- moved U3 81.3 mm to (114.8, 64.6)
- moved C4 81.3 mm to (104.9, 60.3)
- moved C8 81.3 mm to (121.9, 61.8)
- moved C9 81.3 mm to (121.9, 67.1)
- moved D4 78.8 mm to (213.4, 61.0), turned to 90 degrees
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