File: pcb-design/Practical Electronics WS2023/Practical Electronics WS2023.kicad_sch (KiCad schematic)
At the start: 37 parts, among them IC1 SN74HCT04DR, J1 PWR Jack, J2 MIDI Input, J3 MIDI Thru out, J4 Conn_01x03, J5 ISP, J6 Switch connector, J7 Switch connector, J8 Switch connector, U1 6N138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

Commit message: Update schematic
Parts:
- IC1: footprint SOIC127P600X175-14N -> Logic gates:SOIC127P600X175-14N
- U2: footprint Package_SO:SOIC-8-1EP_3.9x4.9mm_P1.27mm_EP2.29x3mm -> Package_SO:SOIC-8-1EP_3.9x4.9mm_P1.27mm_EP2.29x3mm_ThermalVias
Changed lines of the file:
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@@
       (effects (font (size 1.27 1.27)))
     )
-    (property "Footprint" "SOIC127P600X175-14N" (at 63.754 149.098 0)
+    (property "Footprint" "Logic gates:SOIC127P600X175-14N" (at 63.754 149.098 0)
       (effects (font (size 1.27 1.27)) (justify left) hide)
     )
@@
       (effects (font (size 1.27 1.27)))
     )
-    (property "Footprint" "Package_SO:SOIC-8-1EP_3.9x4.9mm_P1.27mm_EP2.29x3mm" (at 213.36 83.82 0)
-      (effects (font (size 1.27 1.27)) (justify left) hide)
-    )
+    (property "Footprint" "Package_SO:SOIC-8-1EP_3.9x4.9mm_P1.27mm_EP2.29x3mm_ThermalVias" (at 213.36 83.82 0)
+      (effects (font (size 1.27 1.27)) (justify left) hide)
+    )

Commit message: PCB WIP
Parts:
- U1: value 6N138 -> 6N138 Optocoupler
- U2: value ADP2303ARDZ-5.0 -> Convertor ADP2303ARDZ-5.0
Changed lines of the file:
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@@
       (effects (font (size 1.27 1.27)))
     )
-    (property "Value" "6N138" (at 211.582 38.608 0)
+    (property "Value" "6N138 Optocoupler" (at 211.582 38.608 0)
       (effects (font (size 1.27 1.27)))
     )
@@
       (effects (font (size 1.27 1.27)))
     )
-    (property "Value" "ADP2303ARDZ-5.0" (at 209.55 64.77 0)
-      (effects (font (size 1.27 1.27)))
-    )
+    (property "Value" "Convertor ADP2303ARDZ-5.0" (at 209.55 64.77 0)
+      (effects (font (size 1.27 1.27)))
+    )
