File: pcb-design/Old/Practical Electronics WS2023/Practical Electronics WS2023.kicad_sch (KiCad schematic)
At the start: 37 parts, among them IC1 SN74HCT04DR, J1 PWR Jack, J2 MIDI Input, J3 MIDI Thru out, J4 Conn_01x03, J5 ISP, J6 Switch connector, J7 Switch connector, J8 Switch connector, U1 6N138 Optocoupler, U2 Convertor ADP2303ARDZ-5.0, U3 ATmega328P-A, Y2 16Mhz

Commit message: Archive old project
Parts:
- added J9: Potentiometer connector, Connector_PinHeader_2.54mm:PinHeader_1x03_P2.54mm_Vertical, symbol Connector_Generic:Conn_01x03
- added R8: 10K, symbol Device:R
- J1: renamed from J6; value Switch connector -> Switch connector 1; footprint Connector_JST:JST_PH_B2B-PH-K_1x02_P2.00mm_Vertical -> Connector_PinHeader_2.54mm:PinHeader_1x02_P2.54mm_Vertical
- J2: renamed from J7; value Switch connector -> Switch connector 2; footprint Connector_JST:JST_PH_B2B-PH-K_1x02_P2.00mm_Vertical -> Connector_PinHeader_2.54mm:PinHeader_1x02_P2.54mm_Vertical
- J7: renamed from J8; value Switch connector -> PWR connector; footprint Connector_JST:JST_PH_B2B-PH-K_1x02_P2.00mm_Vertical -> Connector_PinHeader_2.54mm:PinHeader_1x02_P2.54mm_Vertical
- J8: renamed from J4; value Conn_01x03 -> LED connector; footprint Connector_JST:JST_PH_B3B-PH-K_1x03_P2.00mm_Vertical -> Connector_PinHeader_2.54mm:PinHeader_1x03_P2.54mm_Vertical
- renumbered C1 to C7, C2 to C8, C5 to C9, D18 to D3, H3 to H1, H1 to H2, H2 to H3, J5 to J4, J1 to J5, J2 to J6, R5 to R1, R7 to R2, R2 to R3, R6 to R4, R3 to R5, R4 to R6, R1 to R7, U3 to U1, U1 to U3, Y2 to Y1
Connections:
- net +12V: now also J5.1, J7.2 (Pin_2)
- net +5V: now also J9.1 (Pin_1), R8.1
- net GND: now also J9.3 (Pin_3)
- net RESET: now also R8.2
- net SW: now reaches C8.2, D2.1 (K), L1.1, U2.8 (SW)
- net at U1.9 (PD5): now also J9.2 (Pin_2)
- net ONBOARD LED DATA: no longer names the net of U1.30 (PD0)
Other:
- removed sheet LED circuit
- moved on the sheet: C1, C2, J8, Y1
