File: pcb-design/MIDI visualizer/MIDI visualizer.kicad_pcb (KiCad board)
At the start: 2 copper layers, 68 x 68 mm, 39 parts, among them IC1 SN74HCT04DR, J1 PWR Jack, J2 locked, J3 MIDI Input, J4 MIDI Thru out, J5 Switch 1, J6 Switch 2, J7 Potentiometer, J8 ISP, J9 LED connector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

Commit message: basic traces
Parts:
- moved C7 12.5 mm to (141.2, 72.6), turned to 180 degrees
- moved C6 8.05 mm to (141.2, 75.1), turned to 180 degrees
- moved C8 5.95 mm to (143.3, 89.8), turned to -90 degrees
- moved C9 5.79 mm to (143.3, 82.8), turned to -90 degrees
- moved Y1 5.49 mm to (137.3, 86.4), turned to 90 degrees
- moved C5 4.56 mm to (141.2, 77.5), turned to 180 degrees
- moved R8 0.20 mm to (153.0, 76.6)
Routing:
- net /PGOOD: track 0.00 -> 3.93 mm
- added copper zone on F.Cu, net +5V
- added copper zone on F.Cu, net /SW
- added copper zone on F.Cu, net GND

Commit message: Update pcb
Parts:
- moved J6 16.5 mm to (167.6, 106.6)
- moved J2 13.3 mm to (130.8, 100.2), turned to -90 degrees
- moved R7 13.0 mm to (160.3, 71.9), turned to 90 degrees
- moved R3 12.7 mm to (136.1, 71.0), turned to 0 degrees
- moved J5 8.92 mm to (160.0, 106.6)
- moved C9 8.85 mm to (138.0, 89.9), turned to 0 degrees
- moved C1 8.81 mm to (142.3, 104.0), turned to -90 degrees
- moved C3 8.72 mm to (150.3, 108.1)
- moved Y1 8.52 mm to (141.6, 93.7), turned to 180 degrees
- moved L1 8.39 mm to (153.4, 114.6)
- moved C5 7.50 mm to (143.8, 84.5)
- moved D1 7.12 mm to (146.6, 114.4)
- moved C6 6.26 mm to (143.8, 80.8)
- moved C2 5.84 mm to (141.7, 115.0)
- moved C4 5.73 mm to (133.1, 88.8)
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Routing:
- net +5V: track 0.00 -> 166.8 mm
- net Net-(J4-Pad4): track 0.00 -> 35.8 mm
- net +12V: track 0.00 -> 27.7 mm
- net /SW2 In: track 0.00 -> 26.8 mm, vias 0 -> 2
- net MOSI: track 0.00 -> 26.5 mm, vias 0 -> 2
- net /SW1 In: track 0.00 -> 25.4 mm, vias 0 -> 2
- net MISO: track 0.00 -> 23.2 mm
- net SCK: track 0.00 -> 20.6 mm
- net /Cathode: track 0.00 -> 8.89 mm
- net Net-(J4-Pad5): track 0.00 -> 8.81 mm
- net /Anode: track 0.00 -> 8.22 mm
- net Net-(J2-Pin_1): track 0.00 -> 6.63 mm
- net Net-(IC1-1Y): track 0.00 -> 5.07 mm
- net Net-(J3-Pad4): track 0.00 -> 5.01 mm
- net Net-(D2-K): track 0.00 -> 4.98 mm
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- added copper zone on F.Cu, net +12V
- added copper zone on B.Cu, net GND
Other:
- outline, holes or cut-outs redrawn

Commit message: Polish board
Parts:
- removed J8: ISP, Connector_PinHeader_2.00mm:PinHeader_2x03_P2.00mm_Vertical
- added C10: 0.1uF, Capacitor_SMD:C_1206_3216Metric_Pad1.33x1.80mm_HandSolder, F.Cu at (171.8, 73.9)
- added C11: 1uF, Capacitor_SMD:C_1206_3216Metric_Pad1.33x1.80mm_HandSolder, F.Cu at (157.5, 87.2)
- added J10: UART, Connector_PinSocket_2.54mm:PinSocket_1x06_P2.54mm_Horizontal, B.Cu at (168.8, 79.4)
- H1: value MP1 -> MH; footprint MountingHole:MountingHole_3.2mm_M3_DIN965_Pad_TopBottom -> MountingHole:MountingHole_3.2mm_M3_DIN965
- H2: value MP2 -> MH; footprint MountingHole:MountingHole_3.2mm_M3_DIN965_Pad_TopBottom -> MountingHole:MountingHole_3.2mm_M3_DIN965
- H3: value MP3 -> MH; footprint MountingHole:MountingHole_3.2mm_M3_DIN965_Pad_TopBottom -> MountingHole:MountingHole_3.2mm_M3_DIN965
- H4: value MP4 -> MH; footprint MountingHole:MountingHole_3.2mm_M3_DIN965_Pad_TopBottom -> MountingHole:MountingHole_3.2mm_M3_DIN965
- J7: value Potentiometer -> 1K Pot
- moved J9 24.5 mm to (136.7, 94.9)
- moved R2 15.5 mm to (162.9, 112.6), turned to -90 degrees
- moved J6 15.4 mm to (162.8, 91.9), turned to 0 degrees
- moved R6 13.0 mm to (167.5, 71.0), turned to 90 degrees
- moved J7 12.6 mm to (162.8, 85.3)
- moved Y1 12.2 mm to (132.7, 85.3), turned to 90 degrees
- moved R5 9.41 mm to (118.7, 87.2)
- moved U2 8.59 mm to (120.9, 77.7)
- moved R4 8.54 mm to (122.2, 87.2)
- moved D3 8.32 mm to (121.0, 70.0)
- moved J5 8.07 mm to (162.9, 99.1), turned to 0 degrees
- moved D2 7.79 mm to (159.9, 112.6)
- moved C4 7.57 mm to (125.7, 87.3)
- moved C1 7.34 mm to (135.0, 103.9), turned to 0 degrees
- moved C8 6.95 mm to (136.7, 89.4), turned to -90 degrees
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Connections:
- J1 pad 1: Net-(J2-Pin_1) -> +12V
- J2 pad 1: Net-(J2-Pin_1) -> +12V
- J5 pad 1: /SW1 In -> SW1 In
- J6 pad 1: /SW2 In -> SW2 In
- J7 pad 2: /Pot In -> Pot
- U3 pad 10: /SW1 In -> unconnected-(U3-PD6-Pad10)
- U3 pad 11: /SW2 In -> unconnected-(U3-PD7-Pad11)
- U3 pad 12: MIDI IN -> LED DATA
- U3 pad 13: LED DATA -> unconnected-(U3-PB1-Pad13)
- U3 pad 15: MOSI -> unconnected-(U3-PB3-Pad15)
- U3 pad 16: MISO -> unconnected-(U3-PB4-Pad16)
- U3 pad 17: SCK -> unconnected-(U3-PB5-Pad17)
- U3 pad 23: unconnected-(U3-PC0-Pad23) -> SW1 In
- U3 pad 24: unconnected-(U3-PC1-Pad24) -> SW2 In
- U3 pad 25: unconnected-(U3-PC2-Pad25) -> Pot
- U3 pad 30: unconnected-(U3-PD0-Pad30) -> RX
- U3 pad 31: unconnected-(U3-PD1-Pad31) -> TX
- U3 pad 9: /Pot In -> MIDI IN
Routing:
- net +5V: track 166.8 -> 358.5 mm, vias 0 -> 4
- net MIDI IN: track 3.02 -> 84.9 mm, vias 0 -> 2
- net RESET: track 2.52 -> 58.1 mm
- net RX: track 0.00 -> 51.0 mm, vias 0 -> 2
- net TX: track 0.00 -> 31.6 mm, vias 0 -> 2
- net Net-(J4-Pad4): track 35.8 -> 7.68 mm
- net +12V: track 27.7 -> 0.00 mm
- net /SW2 In: track 26.8 -> 0.00 mm, vias 2 -> 0
- net MOSI: track 26.5 -> 0.00 mm, vias 2 -> 0
- net /SW1 In: track 25.4 -> 0.00 mm, vias 2 -> 0
- net SW1 In: track 0.00 -> 23.6 mm
- net MISO: track 23.2 -> 0.00 mm
- net LED DATA: track 0.00 -> 20.6 mm
- net SCK: track 20.6 -> 0.00 mm
- net SW2 In: track 0.00 -> 17.0 mm
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Other:
- board size 68 x 68 mm -> 68 x 67.9 mm
