File: pcb-design/MIDI visualizer/MIDI visualizer.kicad_sch (KiCad schematic)
At the start: 39 parts, among them IC1 SN74HCT04DR, J1 PWR Jack, J2 PWR connector, J3 MIDI Input, J4 MIDI Thru out, J5 Switch 1, J6 Switch 2, J7 Potentiometer, J8 ISP, J9 LED connector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

Commit message: Polish board
Parts:
- removed H1: MP1, MountingHole:MountingHole_3.2mm_M3_DIN965_Pad_TopBottom, symbol Mechanical:MountingHole_Pad
- removed H2: MP2, MountingHole:MountingHole_3.2mm_M3_DIN965_Pad_TopBottom, symbol Mechanical:MountingHole_Pad
- removed H3: MP3, MountingHole:MountingHole_3.2mm_M3_DIN965_Pad_TopBottom, symbol Mechanical:MountingHole_Pad
- removed H4: MP4, MountingHole:MountingHole_3.2mm_M3_DIN965_Pad_TopBottom, symbol Mechanical:MountingHole_Pad
- removed J8: ISP, Connector_PinHeader_2.00mm:PinHeader_2x03_P2.00mm_Vertical, symbol Connector_Generic:Conn_02x03_Odd_Even
- added C10: 0.1uF, Capacitor_SMD:C_1206_3216Metric_Pad1.33x1.80mm_HandSolder, symbol Device:C
- added C2: 1uF, Capacitor_SMD:C_1206_3216Metric_Pad1.33x1.80mm_HandSolder, symbol Device:C
- added H1, H2, H3, H4: MH, MountingHole:MountingHole_3.2mm_M3_DIN965, symbol Mechanical:MountingHole
- added J10: UART, Connector_PinSocket_2.54mm:PinSocket_1x06_P2.54mm_Horizontal, symbol Connector_Generic:Conn_01x06
- J7: value Potentiometer -> 1K Pot
Connections:
- net +12V: now also J1.1, J2.1 (Pin_1)
- net +5V: now also C2.1, J10.4 (Pin_4)
- net GND: now also C2.2, J10.6 (Pin_6)
- net LED DATA: now also U3.12 (PB0); no longer U3.13 (PB1)
- net MIDI IN: now also U3.9 (PD5); no longer U3.12 (PB0)
- net RESET: now also C10.1, C10.2, J10.1 (Pin_1)
- net SW1 In: now also U3.23 (PC0); no longer U3.10 (PD6)
- net SW2 In: now also U3.24 (PC1); no longer U3.11 (PD7)
- net Pot: now reaches U3.25 (PC2)
- net Pot: now also J7.2 (Pin_2)
- net RX: now reaches U3.30 (PD0)
- net RX: now also J10.3 (Pin_3)
- net TX: now reaches U3.31 (PD1)
- net TX: now also J10.2 (Pin_2)
- net MISO: no longer names the net of U3.16 (PB4)
- net MOSI: no longer names the net of U3.15 (PB3)
- removed net Pot In: J7.2 (Pin_2), U3.9 (PD5)
- net SCK: no longer names the net of U3.17 (PB5)
- no-connect marks 28 -> 30
Other:
- note added: "UART programmer"
- note removed: "ISP"
- moved on the sheet: C1, C2, C3, D1, D2, J1, J2, J5, J6, J7, J9, L1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
